File: mfm-v3-smd.kicad_sch (KiCad schematic)
At the start: 47 parts, among them J1 MFM Module-Left, J2 MFM Module-Right, J3 SMBUS Connector, J4 FTDI Connector, J5 ICSP Connector, J6 Antenna, J7 JST Jack, Q1 R.V. Protect, SW1 SW_VBAT, SW2 RESET, SW3 SW_LED_PWR, SW4 SW_LED_STAT, U1 MCP1703A-3302_SOT89, U2 LoRa_Radio, U3 ATmega1284P-AU, Y1 8MHz

Commit message: initial setup of v3.7
Parts:
- removed BT1: Battery, Battery:BatteryHolder_Keystone_2462_2xAA, symbol Device:Battery
- removed C12: 820uF 16v, Capacitor_SMD:C_Elec_8x10.2, symbol Device:CP_Small
- removed J1: MFM Module-Left, custom_library_FP:MFM_Module_Board_P123, symbol Connector_Generic:Conn_01x03
- removed J2: MFM Module-Right, Connector_PinSocket_2.54mm:PinSocket_1x03_P2.54mm_Vertical, symbol Connector_Generic:Conn_01x03
- removed J3: SMBUS Connector, Connector_PinHeader_2.54mm:PinHeader_2x03_P2.54mm_Vertical, symbol Connector_Generic:Conn_02x03_Odd_Even
- removed J4: FTDI Connector, Connector_PinSocket_2.54mm:PinSocket_1x06_P2.54mm_Vertical, symbol Connector_Generic:Conn_01x06
- removed J5: ICSP Connector, Connector_PinHeader_2.54mm:PinHeader_2x03_P2.54mm_Vertical, symbol Connector_Generic:Conn_02x03_Odd_Even
- removed R6, R9: 4k7, custom_library_FP:R_0603_1608Metric_CRCW...C, symbol Device:R_Small
- removed SW3: SW_LED_PWR, Connector_PinHeader_2.54mm:PinHeader_1x02_P2.54mm_Vertical, symbol Switch:SW_SPST
- removed SW4: SW_LED_STAT, Connector_PinHeader_2.54mm:PinHeader_1x02_P2.54mm_Vertical, symbol Switch:SW_SPST
- removed U1: MCP1703A-3302_SOT89, custom_library_FP:SOT-89-3_MCP1703, symbol Regulator_Linear:MCP1703A-3302_SOT89
- removed U3: ATmega1284P-AU, Package_QFP:TQFP-44_10x10mm_P0.8mm, symbol MCU_Microchip_ATmega:ATmega1284P-AU
- added IC1: AP7370-33Y, Package_TO_SOT_SMD:SOT-89-3, symbol custom_library:AP7370-33Y
- added J1: JST Jack, Connector_JST:JST_PH_B2B-PH-SM4-TB_1x02-1MP_P2.00mm_Vertical, symbol mfm-v3-smd-rescue:JST_Jack-Connector
- added J4: MFM Module connector, Connector_JST:JST_PH_B7B-PH-SM4-TB_1x07-1MP_P2.00mm_Vertical, symbol custom_library:MFM Module connector
- added JP1: SW_LED_PWR, Jumper:SolderJumper-2_P1.3mm_Open_RoundedPad1.0x1.5mm, symbol Jumper:Jumper_2_Open
- added JP2: SW_LED_STAT, Jumper:SolderJumper-2_P1.3mm_Open_RoundedPad1.0x1.5mm, symbol Jumper:Jumper_2_Open
- added P1: AVR-JTAG-10-TC2050(non-reversed), Tag-Connect_footprints:TC2050-IDC-NL, symbol Tag-Connect:AVR-JTAG-10-TC2050(non-reversed)
- added Q2: R.V. Protect, Package_TO_SOT_SMD:SOT-23, symbol Device:Q_PMOS_GSD
- added TP1: GND, TestPoint:TestPoint_Pad_D1.5mm, symbol Connector:TestPoint
- added TP2: TX0, TestPoint:TestPoint_Pad_D1.5mm, symbol Connector:TestPoint
- added U1: ATmega1284P-M, Package_DFN_QFN:QFN-44-1EP_7x7mm_P0.5mm_EP5.2x5.2mm, symbol MCU_Microchip_ATmega:ATmega1284P-M
- J2: renamed from J7; footprint Connector_JST:JST_XH_B2B-XH-A_1x02_P2.50mm_Vertical -> Connector_JST:JST_PH_B2B-PH-SM4-TB_1x02-1MP_P2.00mm_Vertical
- J3: renamed from J6; footprint custom_library_FP:LINX_CONSMA001-SMD-G -> CONMHF1-SMD-G-T:LINX_CONMHF1-SMD-G-T
- SW2: footprint custom_library_FP:SW_SPST_PTS636 -> PTS815-SJK-250-SMTR-LFS:PTS815SJK250SMTRLFS
- renumbered R8 to R6
Connections:
- net +3V3: now also IC1.1 (Vout), J4.1 (+3V3), P1.4 (VTG/VCC), U1.17 (VCC), U1.27 (AVCC), U1.38 (VCC), U1.5 (VCC)
- net AVR_MISO: now also P1.3 (TDO), U1.2 (PB6)
- net AVR_MOSI: now also U1.1 (PB5)
- net AVR_RX0: now also U1.9 (PD0)
- net AVR_RX1: now also U1.11 (PD2)
- net AVR_SCK: now also P1.1 (TCK), U1.3 (PB7)
- net AVR_TX0: now also TP2.1, U1.10 (PD1)
- net AVR_TX1: now also U1.12 (PD3)
- net GND: now also IC1.2 (GND), J1.1, J4.4 (GND), JP1.2 (B), JP2.2 (B), P1.10 (GND), P1.2 (GND), Q2.1 (G), TP1.1, U1.18 (GND), U1.28 (GND), U1.39 (GND), U1.45 (GND), U1.6 (GND)
- net I2C_SCL: now also J4.3 (SCL), U1.19 (PC0)
- net I2C_SDA: now also J4.6 (SDA), U1.20 (PC1)
- net LED_STAT: now also U1.34 (PA3)
- net NRST: now also P1.6 (~{SRST}), U1.4 (~{RESET})
- net RADIO_DIO0: now also U1.42 (PB2)
- net RADIO_DIO1: now also U1.43 (PB3)
- net RADIO_DIO2: now also U1.44 (PB4)
- net RADIO_DIO3: now also U1.40 (PB0)
- net RADIO_DIO4: now also U1.41 (PB1)
- net RADIO_DIO5: now also U1.35 (PA2)
- net RADIO_NSS: now also U1.37 (PA0)
- net RADIO_RST: now also U1.36 (PA1)
- net SMBALERT: now also J4.5 (SMB_Alert), U1.21 (PC2)
- net SPI_MOSI: now also P1.9 (TDI)
- net VBAT: now also C1.2, IC1.3 (Vin), J4.2 (+VBat); no longer Q1.3 (D)
- net XTAL1: now also U1.8 (XTAL1)
- net XTAL2: now also U1.7 (XTAL2)
- net at C11.2: now also U1.29 (AREF)
- net RV_Protect: now reaches Q1.2 (S)
- net RV_Protect: now also SW1.1 (A), Q2.2 (S); no longer C1.2
- net Bat_in_1: now reaches J2.2
- net Bat_in_1: now also Q1.3 (D); no longer SW1.1 (A)
- net at D1.1 (K): now also JP1.1 (A)
- net at D2.1 (K): now also JP2.1 (A)
- new net Bat_in_2: J1.2, Q2.3 (D)
Other:
- note added: "FTDI Debug"
- note added: "LED POWER = Blue Vf = 2.65 V If = 2 mA Lum = 50 mcd R = (3.3V-2.65V) / 2mA = 325Ω"
- note added: "PSU"
- note removed: "3.3V Power supply"
- note removed: "Battery pins"
- note removed: "FTDI Connector"
- note removed: "LED POWER = BLUE Vf = 2.65 V If = 2 mA Lum = 50 mcd R = (3.3V-2.65V) / 2mA = 325Ω"
- note removed: "SMBUS Connector"
- moved on the sheet: C1, C2, C5, C7, C8, D1, D2, J2, J3, Q1, R1, R2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
